File: Pi-BLDC-Controller/Pi-BLDC-Controller.kicad_sch (KiCad schematic)
At the start: 1 part, among them U1 RP2040

Commit message: all
Parts:
- removed U1: RP2040, Package_DFN_QFN:QFN-56-1EP_7x7mm_P0.4mm_EP3.2x3.2mm, symbol MCU_RaspberryPi:RP2040
- added C1, C19, C5: 10u, Capacitor_SMD:C_0805_2012Metric, symbol MCU_RaspberryPi_RP2350:C
- added C10, C9: 4.7u, Capacitor_SMD:C_0402_1005Metric, symbol MCU_RaspberryPi_RP2350:C
- added C11, C12, C13, C14, C15, C16, C17, C18, C2, C8: 100n, Capacitor_SMD:C_0402_1005Metric, symbol MCU_RaspberryPi_RP2350:C
- added C20: 1000pF, symbol MCU_RaspberryPi_RP2350:C
- added C21, C22: 1000pF, Capacitor_SMD:C_0603_1608Metric_Pad1.08x0.95mm_HandSolder, symbol MCU_RaspberryPi_RP2350:C
- added C23, C24, C25: 1uF 100V, Diode_SMD:D_1206_3216Metric_Pad1.42x1.75mm_HandSolder, symbol MCU_RaspberryPi_RP2350:C
- added C3, C4: 15p, Capacitor_SMD:C_0402_1005Metric, symbol MCU_RaspberryPi_RP2350:C
- added C6, C7: 4.7u, RP2350_60QFN_minimal:C_0402_1005Metric_small_pads, symbol MCU_RaspberryPi_RP2350:C
- added J1: USB_B_Micro, Connector_USB:USB_Micro-B_Amphenol_10103594-0001LF_Horizontal, symbol MCU_RaspberryPi_RP2350:USB_B_Micro
- added J2: Conn_01x03, symbol Connector_Generic:Conn_01x03
- added J4: SM03B-SRSS-TB, Connector_JST:JST_SH_SM03B-SRSS-TB_1x03-1MP_P1.00mm_Horizontal, symbol MCU_RaspberryPi_RP2350:Conn_01x03_MountingPin
- added L1: 3.3u, RP2350_60QFN_minimal:L_pol_2016, symbol MCU_RaspberryPi_RP2350:L
- added Q1, Q2, Q3, Q4, Q5, Q6: SIR680LDP, Package_SO:PowerPAK_SO-8_Single, symbol Transistor_FET:SiR696DP
- added R1, R9: DNF, Resistor_SMD:R_0402_1005Metric, symbol MCU_RaspberryPi_RP2350:R
- added R10: 0, Resistor_SMD:R_0402_1005Metric, symbol MCU_RaspberryPi_RP2350:R
- added R11: 10k, symbol MCU_RaspberryPi_RP2350:R
- added R12, R13, R14: 0.007 Ohm, Resistor_SMD:R_2512_6332Metric_Pad1.40x3.35mm_HandSolder, symbol MCU_RaspberryPi_RP2350:R
- added R2, R4, R6: 1k, Resistor_SMD:R_0402_1005Metric, symbol MCU_RaspberryPi_RP2350:R
- added R3: 1k, symbol MCU_RaspberryPi_RP2350:R
- added R5: 33, Resistor_SMD:R_0402_1005Metric, symbol MCU_RaspberryPi_RP2350:R
- added R7, R8: 27, Resistor_SMD:R_0402_1005Metric, symbol MCU_RaspberryPi_RP2350:R
- added SW1, SW2: SW_Push, Button_Switch_SMD:SW_Push_1P1T_NO_Vertical_Wuerth_434133025816, symbol MCU_RaspberryPi_RP2350:SW_Push
- added U1: RP2350_60QFN, RP2350_60QFN_minimal:RP2350-QFN-60-1EP_7x7_P0.4mm_EP3.4x3.4mm_ThermalVias, symbol MCU_RaspberryPi_RP2350:RP2350_60QFN
- added U2: NCP1117-3.3_SOT223, Package_TO_SOT_SMD:SOT-223-3_TabPin2, symbol MCU_RaspberryPi_RP2350:NCP1117-3.3_SOT223
- added U3: W25Q128JVS, Package_SO:SOIC-8_5.23x5.23mm_P1.27mm, symbol MCU_RaspberryPi_RP2350:W25Q128JVS
- added U4: DRV8353RHRGZR, RGZ0048L, symbol 2025-07-07_14-36-57:DRV8353RHRGZR
- added Y1: ABM8-272-T3, Crystal:Crystal_SMD_3225-4Pin_3.2x2.5mm, symbol MCU_RaspberryPi_RP2350:Crystal_GND24
Connections:
- new net: R7.2, U1.52 (USB_DP)
- new net: R8.2, U1.51 (USB_DM)
- new net: R4.1, SW2.1
- new net: C4.1, R2.2, Y1.3
- new net +1V1: C10.1, C11.1, C7.1, C8.1, L1.1, U1.23 (DVDD), U1.39 (DVDD), U1.50 (VREG_FB), U1.6 (DVDD)
- new net +3V3: C12.1, C13.1, C14.1, C15.1, C16.1, C17.1, C18.1, C19.1, C2.1, C5.1, C6.1, R1.1, R11.1, R3.1, R5.1, U1.1 (IOVDD), U1.11 (IOVDD), U1.20 (IOVDD), U1.30 (IOVDD), U1.38 (IOVDD), U1.44 (ADC_AVDD), U1.45 (IOVDD), U1.49 (VREG_VIN), U1.53 (USB_OTP_VDD), U1.54 (QSPI_IOVDD), U2.2 (VO), U3.8 (VCC)
- new net DRV_EN: U4.33 (ENABLE)
- new net DRV_SCLK: U1.4 (GPIO2), U4.31 (VDS_SCLK)
- new net DRV_SDI: U1.5 (GPIO3), U4.30 (IDRIVE_SDI)
- new net DRV_SDO: R3.2, R9.1, U1.2 (GPIO0), U4.29 (MODE_SDO)
- new net DRV_nFAULT: R11.2, U4.28 (FAULT_N)
- new net DRV_nSCS: U1.3 (GPIO1), U4.32 (NC_SCS_N)
- new net FLASH_SS: R1.2, R10.2, R9.2, U3.1 (~{CS})
- new net GHA: Q1.4 (G), U4.8 (GHA)
- new net GHB: Q3.4 (G), U4.17 (GHB)
- new net GHC: Q5.4 (G), U4.18 (GHC)
- new net GLA: Q2.4 (G), U4.10 (GLA)
- new net GLB: Q4.4 (G), U4.15 (GLB)
- new net GLC: Q6.4 (G), U4.20 (GLC)
- new net GND: C1.2, C10.2, C11.2, C12.2, C13.2, C14.2, C15.2, C16.2, C17.2, C18.2, C19.2, C2.2, C20.2, C21.2, C22.2, C23.2, C24.2, C25.2, C3.2, C4.2, C5.2, C6.2, C7.2, C8.2, C9.2, J1.5 (GND), J1.6 (Shield), J4.2 (Pin_2), J4.MP (MountPin), R12.2, R13.2, R14.2, R4.2, SW1.1, U1.47 (VREG_PGND), U1.61 (GND), U2.1 (GND), U3.4 (GND), U4.12 (SNA), U4.13 (SNB), U4.22 (SNC), U4.38 (INHC), Y1.2, Y1.4
- new net GPIO10: U1.14 (GPIO10)
- new net GPIO11: U1.15 (GPIO11)
- new net GPIO12: U1.16 (GPIO12)
- new net GPIO13: U1.17 (GPIO13)
- new net GPIO14: U1.18 (GPIO14)
- new net GPIO15: U1.19 (GPIO15)
- new net GPIO16: U1.27 (GPIO16)
- new net GPIO17: U1.28 (GPIO17)
- new net GPIO18: U1.29 (GPIO18)
- new net GPIO19: U1.31 (GPIO19)
- new net GPIO20: U1.32 (GPIO20)
- new net GPIO21: U1.33 (GPIO21)
- new net GPIO22: U1.34 (GPIO22)
- new net GPIO23: U1.35 (GPIO23)
- new net GPIO24: U1.36 (GPIO24)
- new net GPIO25: U1.37 (GPIO25)
- new net GPIO26_ADC0: U1.40 (GPIO26_ADC0)
- new net GPIO27_ADC1: U1.41 (GPIO27_ADC1)
- new net GPIO28_ADC2: U1.42 (GPIO28_ADC2)
- new net GPIO29_ADC3: U1.43 (GPIO29_ADC3)
- new net GPIO4: U1.7 (GPIO4)
- new net GPIO5: U1.8 (GPIO5)
- new net GPIO6: U1.9 (GPIO6)
- new net GPIO7: U1.10 (GPIO7)
- new net GPIO8: U1.12 (GPIO8)
- new net GPIO9: U1.13 (GPIO9)
- new net HALL_A: U4.35 (INLA)
- new net HALL_B: U4.36 (INHB)
- new net HALL_C: U4.37 (INLB)
- new net MCU_PWM: U4.34 (INHA)
- new net MOTA: J2.1 (Pin_1), Q1.1 (S), Q1.2 (S), Q1.3 (S), Q2.5 (D), U4.9 (SHA)
- new net MOTB: J2.2 (Pin_2), Q3.1 (S), Q3.2 (S), Q3.3 (S), Q4.5 (D), U4.16 (SHB)
- new net MOTC: J2.3 (Pin_3), Q5.1 (S), Q5.2 (S), Q5.3 (S), Q6.5 (D), U4.19 (SHC)
- new net QSPI_SCLK: U1.56 (QSPI_SCLK), U3.6 (CLK)
- new net QSPI_SD0: U1.57 (QSPI_SD0), U3.5 (DI(IO0))
- new net QSPI_SD1: U1.59 (QSPI_SD1), U3.2 (DO(IO1))
- new net QSPI_SD2: U1.58 (QSPI_SD2), U3.3 (IO2)
- new net QSPI_SD3: U1.55 (QSPI_SD3), U3.7 (IO3)
- new net QSPI_SS: R10.1, R6.1, U1.60 (QSPI_SS)
- new net RUN: SW2.2, U1.26 (RUN)
- new net SPA: C20.1, Q2.1 (S), Q2.2 (S), Q2.3 (S), R12.1, U4.11 (SPA)
- new net SPB: C21.1, Q4.1 (S), Q4.2 (S), Q4.3 (S), R13.1, U4.14 (SPB)
- new net SPC: C22.1, Q6.1 (S), Q6.2 (S), Q6.3 (S), R14.1, U4.21 (SPC)
- new net SWCLK: J4.1 (Pin_1), U1.24 (SWCLK)
- new net SWD: J4.3 (Pin_3), U1.25 (SWD)
- new net USB_D+: J1.3 (D+), R7.1
- new net USB_D-: J1.2 (D-), R8.1
- new net VBUS: C1.1, J1.1 (VBUS), U2.3 (VI)
- new net VDRAIN: U4.6 (VDRAIN)
- new net VM: C23.1, C24.1, C25.1, Q1.5 (D), Q3.5 (D), Q5.5 (D)
- new net VREG_AVDD: C9.1, R5.2, U1.46 (VREG_AVDD)
- new net VREG_LX: L1.2, U1.48 (VREG_LX)
- new net XIN: C3.1, U1.21 (XIN), Y1.1
- new net XOUT: R2.1, U1.22 (XOUT)
- new net nBRAKE: U4.39 (INLC)
- new net ~{USB_BOOT}: R6.2, SW1.2
- no-connect marks 0 -> 1
Other:
- note added: "12MHz Crystal"
- note added: "CBYP"
- note added: "Flash"
- note added: "JST Debug Connector"
- note added: "Make sure R7 and R8 are close to RP2350"
- note added: "No direction control"
- note added: "Power"
- note added: "pull-up resistor."

Commit message: all
Parts:
- added C26: 1uF, Capacitor_SMD:C_1206_3216Metric_Pad1.33x1.80mm_HandSolder, symbol MCU_RaspberryPi_RP2350:C
- added J3: Conn_01x05, symbol Connector_Generic:Conn_01x05
- added R15, R16, R17: 1k, symbol MCU_RaspberryPi_RP2350:R
Connections:
- net +3V3: now also R15.1, R16.1, R17.1
- net GND: now also J3.5 (Pin_5); no longer U4.38 (INHC)
- net HALL_B: now also J3.3 (Pin_3), R16.2; no longer U4.36 (INHB)
- net HALL_C: now also J3.2 (Pin_2), J3.4 (Pin_4), R15.2, R17.2; no longer U4.37 (INLB)
- net at U4.5 (VM): now also C26.1
- net at U4.7 (VCP): now also C26.2
- net HALL_A renamed DRV_GLA
- net MCU_PWM renamed DRV_GHA
- net nBRAKE renamed DRV_GLC
- new net +12V: J3.1 (Pin_1)
- new net DRV_GHB: U4.36 (INHB)
- new net DRV_GHC: U4.38 (INHC)
- new net DRV_GLB: U4.37 (INLB)
Other:
- note added: "6x PWM Mode"
- note added: "Filter"
- note removed: "No direction control"
- moved on the sheet: J2, R11, R3
