File: slvc742a/MD016A Design Files/MD016A.kicad_sch (KiCad schematic)
At the start: 150 parts, among them J1 SSQ-110-01-G-D-001-LL, J2 SSQ-110-01-G-D, J3 1792892, J5 1902547, J6 1904150, Q1 CSD19532Q5B, Q2 CSD19532Q5B, Q3 CSD19532Q5B, Q4 CSD19532Q5B, Q5 CSD19532Q5B, Q6 CSD19532Q5B, U1 TPD4S010DQAR, U2 DRV8353RSRGZR, U3 LP2992IM5-3.3/NOPB

Commit message: all
Other:
- note removed: "Filter Cap"
